File: kicad/prilkeeb.kicad_sch (KiCad schematic)
At the start: 73 parts, among them U2 Nice_Nano_V2

Commit message: Update MCU position
Connections:
- net Col_1: now also S13.1, S20.1, S27.1, S30.1, S6.1, U2.14 (16); no longer S12.1, S19.1, S26.1, S29.1, S5.1, U2.20 (21)
- net Col_2: now also S1.1, S15.1, S22.1, S31.1, S8.1, U2.15 (14); no longer S13.1, S20.1, S27.1, S30.1, S6.1, U2.19 (20)
- net Col_3: now also S16.1, S2.1, S23.1, S35.1, S9.1, U2.16 (15); no longer S1.1, S15.1, S22.1, S31.1, S8.1, U2.18 (19)
- net Col_4: now also S10.1, S17.1, S24.1, S3.1, S32.1; no longer S16.1, S2.1, S23.1, S35.1, S9.1
- net Col_5: now also S11.1, S18.1, S25.1, S33.1, S4.1, U2.18 (19); no longer S10.1, S17.1, S24.1, S3.1, S32.1, U2.16 (15)
- net Col_6: now also S14.1, S21.1, S28.1, S34.1, S7.1, U2.19 (20); no longer S11.1, S18.1, S25.1, S33.1, S4.1, U2.15 (14)
- net Row_1: now also D10.1 (K), D11.1 (K), D12.1 (K), D13.1 (K), D14.1 (K), D8.1 (K), D9.1 (K), U2.9 (6); no longer D1.1 (K), D2.1 (K), D3.1 (K), D4.1 (K), D5.1 (K), D6.1 (K), D7.1 (K), U2.5 (2)
- net Row_2: now also D15.1 (K), D16.1 (K), D17.1 (K), D18.1 (K), D19.1 (K), D20.1 (K), D21.1 (K), U2.10 (7); no longer D10.1 (K), D11.1 (K), D12.1 (K), D13.1 (K), D14.1 (K), D8.1 (K), D9.1 (K), U2.6 (3)
- net Row_3: now also D22.1 (K), D23.1 (K), D24.1 (K), D25.1 (K), D26.1 (K), D27.1 (K), D28.1 (K), U2.11 (8); no longer D15.1 (K), D16.1 (K), D17.1 (K), D18.1 (K), D19.1 (K), D20.1 (K), D21.1 (K), U2.7 (4)
- net Row_4: now also D29.1 (K), D30.1 (K), D31.1 (K), D32.1 (K), D33.1 (K), D34.1 (K), D35.1 (K), U2.12 (9); no longer D22.1 (K), D23.1 (K), D24.1 (K), D25.1 (K), D26.1 (K), D27.1 (K), D28.1 (K), U2.8 (5)
- net Col_0: now reaches U2.13 (10)
- net Col_0: now also S12.1, S19.1, S26.1, S29.1, S5.1
- removed net Col_7: S14.1, S21.1, S28.1, S34.1, S7.1, U2.14 (16)
- removed net Row_5: D29.1 (K), D30.1 (K), D31.1 (K), D32.1 (K), D33.1 (K), D34.1 (K), D35.1 (K), U2.9 (6)
- new net Row_0: D1.1 (K), D2.1 (K), D3.1 (K), D4.1 (K), D5.1 (K), D6.1 (K), D7.1 (K), U2.8 (5)
