File: kicad/prilkeeb.kicad_sch (KiCad schematic)
At the start: 75 parts, among them SW1 SW_SPDT, U2 Nice_Nano_V2

Commit message: Update diode type
Parts:
- D1, D10, D11, D12, D13, D14, D15, D16, D17, D18, D19, D2, D20, D21, D22, D23, D24, D25, D26, D27, D28, D29, D3, D30, D31, D32, D33, D34, D4, D5, D6, D7, D8, D9, DROTARY1: footprint ScottoKeebs_Components:Diode_DO-35 -> dumta:D_SMD_TH
Changed lines of the file:
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@@
 			)
 		)
-		(property "Footprint" "ScottoKeebs_Components:Diode_DO-35"
+		(property "Footprint" "dumta:D_SMD_TH"
 			(at 69.85 109.22 90)
 			(effects
@@
 			)
 		)
-		(property "Footprint" "ScottoKeebs_Components:Diode_DO-35"
+		(property "Footprint" "dumta:D_SMD_TH"
 			(at 41.91 124.46 90)
 			(effects
@@
 			)
 		)
-		(property "Footprint" "ScottoKeebs_Components:Diode_DO-35"
+		(property "Footprint" "dumta:D_SMD_TH"
 			(at 55.88 93.98 90)
 			(effects
@@
 			)
 		)
-		(property "Footprint" "ScottoKeebs_Components:Diode_DO-35"
+		(property "Footprint" "dumta:D_SMD_TH"
 			(at 114.3 139.7 90)
 			(effects
@@
 			)
 		)
-		(property "Footprint" "ScottoKeebs_Components:Diode_DO-35"
+		(property "Footprint" "dumta:D_SMD_TH"
 			(at 99.06 109.22 90)
 			(effects
@@
 			)
 		)
-		(property "Footprint" "ScottoKeebs_Components:Diode_DO-35"
+		(property "Footprint" "dumta:D_SMD_TH"
 			(at 69.85 124.46 90)
 			(effects
@@
 			)
 		)
-		(property "Footprint" "ScottoKeebs_Components:Diode_DO-35"
+		(property "Footprint" "dumta:D_SMD_TH"
 			(at 128.27 93.98 90)
 			(effects
@@
 			)
 		)
-		(property "Footprint" "ScottoKeebs_Components:Diode_DO-35"
+		(property "Footprint" "dumta:D_SMD_TH"
 			(at 114.3 109.22 90)
 			(effects
@@
 			)
 		)
-		(property "Footprint" "ScottoKeebs_Components:Diode_DO-35"
+		(property "Footprint" "dumta:D_SMD_TH"
 			(at 114.3 124.46 90)
 			(effects
@@
 			)
 		)
-		(property "Footprint" "ScottoKeebs_Components:Diode_DO-35"
+		(property "Footprint" "dumta:D_SMD_TH"
 			(at 128.27 78.74 90)
 			(effects
@@
 			)
 		)
-		(property "Footprint" "ScottoKeebs_Components:Diode_DO-35"
+		(property "Footprint" "dumta:D_SMD_TH"
 			(at 83.82 124.46 90)
 			(effects
@@
 			)
 		)
-		(property "Footprint" "ScottoKeebs_Components:Diode_DO-35"
+		(property "Footprint" "dumta:D_SMD_TH"
 			(at 41.91 139.7 90)
 			(effects
@@
 			)
 		)
-		(property "Footprint" "ScottoKeebs_Components:Diode_DO-35"
+		(property "Footprint" "dumta:D_SMD_TH"
 			(at 41.91 109.22 90)
 			(effects
@@
 			)
 		)
-		(property "Footprint" "ScottoKeebs_Components:Diode_DO-35"
+		(property "Footprint" "dumta:D_SMD_TH"
 			(at 69.85 139.7 90)
 			(effects
@@
 			)
 		)
-		(property "Footprint" "ScottoKeebs_Components:Diode_DO-35"
+		(property "Footprint" "dumta:D_SMD_TH"
 			(at 55.88 124.46 90)
 			(effects
@@
 			)
 		)
-		(property "Footprint" "ScottoKeebs_Components:Diode_DO-35"
+		(property "Footprint" "dumta:D_SMD_TH"
 			(at 128.27 124.46 90)
 			(effects
@@
 			)
 		)
-		(property "Footprint" "ScottoKeebs_Components:Diode_DO-35"
+		(property "Footprint" "dumta:D_SMD_TH"
 			(at 55.88 78.74 90)
 			(effects
@@
 			)
 		)
-		(property "Footprint" "ScottoKeebs_Components:Diode_DO-35"
+		(property "Footprint" "dumta:D_SMD_TH"
 			(at 114.3 93.98 90)
 			(effects
@@
 			)
 		)
-		(property "Footprint" "ScottoKeebs_Components:Diode_DO-35"
+		(property "Footprint" "dumta:D_SMD_TH"
 			(at 41.91 78.74 90)
 			(effects
@@
 			)
 		)
-		(property "Footprint" "ScottoKeebs_Components:Diode_DO-35"
+		(property "Footprint" "dumta:D_SMD_TH"
 			(at 41.91 93.98 90)
 			(effects
@@
 			)
 		)
-		(property "Footprint" "ScottoKeebs_Components:Diode_DO-35"
+		(property "Footprint" "dumta:D_SMD_TH"
 			(at 83.82 93.98 90)
 			(effects
@@
 			)
 		)
-		(property "Footprint" "ScottoKeebs_Components:Diode_DO-35"
+		(property "Footprint" "dumta:D_SMD_TH"
 			(at 83.82 139.7 90)
 			(effects
@@
 			)
 		)
-		(property "Footprint" "ScottoKeebs_Components:Diode_DO-35"
+		(property "Footprint" "dumta:D_SMD_TH"
 			(at 55.88 109.22 90)
 			(effects
@@
 			)
 		)
-		(property "Footprint" "ScottoKeebs_Components:Diode_DO-35"
+		(property "Footprint" "dumta:D_SMD_TH"
 			(at 99.06 139.7 90)
 			(effects
@@
 			)
 		)
-		(property "Footprint" "ScottoKeebs_Components:Diode_DO-35"
+		(property "Footprint" "dumta:D_SMD_TH"
 			(at 128.27 139.7 90)
 			(effects
@@
 			)
 		)
-		(property "Footprint" "ScottoKeebs_Components:Diode_DO-35"
+		(property "Footprint" "dumta:D_SMD_TH"
 			(at 99.06 124.46 90)
 			(effects
@@
 			)
 		)
-		(property "Footprint" "ScottoKeebs_Components:Diode_DO-35"
+		(property "Footprint" "dumta:D_SMD_TH"
 			(at 114.3 78.74 90)
 			(effects
@@
 			)
 		)
-		(property "Footprint" "ScottoKeebs_Components:Diode_DO-35"
+		(property "Footprint" "dumta:D_SMD_TH"
 			(at 99.06 93.98 90)
 			(effects
@@
 			)
 		)
-		(property "Footprint" "ScottoKeebs_Components:Diode_DO-35"
+		(property "Footprint" "dumta:D_SMD_TH"
 			(at 69.85 93.98 90)
 			(effects
@@
 			)
 		)
-		(property "Footprint" "ScottoKeebs_Components:Diode_DO-35"
+		(property "Footprint" "dumta:D_SMD_TH"
 			(at 128.27 109.22 90)
 			(effects
@@
 			)
 		)
-		(property "Footprint" "ScottoKeebs_Components:Diode_DO-35"
+		(property "Footprint" "dumta:D_SMD_TH"
 			(at 69.85 78.74 90)
 			(effects
@@
 			)
 		)
-		(property "Footprint" "ScottoKeebs_Components:Diode_DO-35"
+		(property "Footprint" "dumta:D_SMD_TH"
 			(at 83.82 78.74 90)
 			(effects
@@
 			)
 		)
-		(property "Footprint" "ScottoKeebs_Components:Diode_DO-35"
+		(property "Footprint" "dumta:D_SMD_TH"
 			(at 99.06 78.74 90)
 			(effects
@@
 			)
 		)
-		(property "Footprint" "ScottoKeebs_Components:Diode_DO-35"
+		(property "Footprint" "dumta:D_SMD_TH"
 			(at 55.88 139.7 90)
 			(effects
@@
 			)
 		)
-		(property "Footprint" "ScottoKeebs_Components:Diode_DO-35"
+		(property "Footprint" "dumta:D_SMD_TH"
 			(at 83.82 109.22 90)
 			(effects
